File: power-supply.kicad_pcb (KiCad board)
At the start: 2 copper layers, 101.6 x 38.1 mm, 22 parts, among them J1 AC, J2 DC, M1 MountingHole_2.2mm_M2, M2 MountingHole_2.2mm_M2, M3 MountingHole_2.2mm_M2, M4 MountingHole_2.2mm_M2, U1 LM7815_TO220, U2 LM7915_TO220

Commit message: update: update file
Parts:
- added REF**: OSHW-Logo2_9.8x8mm_SilkScreen, Symbol:OSHW-Logo2_9.8x8mm_SilkScreen, F.Cu at (114.3, 87.6)
Routing:
- net GND: track 181.6 -> 183.7 mm
