File: power-supply.sch (KiCad schematic (older format))
At the start: 18 parts, among them J1 AC, J2 DC, U1 LM7815_TO220, U2 LM7915_TO220

Commit message: update
I changed the value of the resistors to a more satisfactory one
Parts:
- R1, R2: value 330R -> 1k3
Changed lines of the file:
@@
 P 7650 2850
 F 0 "R1" H 7720 2896 50  0000 L CNN
-F 1 "330R" H 7720 2805 50  0000 L CNN
+F 1 "1k3" H 7720 2805 50  0000 L CNN
 F 2 "Resistor_THT:R_Axial_DIN0207_L6.3mm_D2.5mm_P5.08mm_Vertical" V 7580 2850 50  0001 C CNN
 F 3 "~" H 7650 2850 50  0001 C CNN
@@
 P 7650 3850
 F 0 "R2" H 7720 3896 50  0000 L CNN
-F 1 "330R" H 7720 3805 50  0000 L CNN
+F 1 "1k3" H 7720 3805 50  0000 L CNN
 F 2 "Resistor_THT:R_Axial_DIN0207_L6.3mm_D2.5mm_P5.08mm_Vertical" V 7580 3850 50  0001 C CNN
 F 3 "~" H 7650 3850 50  0001 C CNN
